File: dcdc.sch (KiCad schematic (older format))
At the start: 0 parts

Commit message: dcdc доделан на 5V.
Parts:
- added C31: 100uF, Capacitor_SMD:C_1206_3216Metric_Pad1.42x1.75mm_HandSolder, symbol Device:C
- added C32: 10uF, Capacitor_SMD:C_1206_3216Metric_Pad1.42x1.75mm_HandSolder, symbol Device:C
- added C33: 100nF, Capacitor_SMD:C_0805_2012Metric_Pad1.15x1.40mm_HandSolder, symbol Device:C
- added D6: 1N5819, Diode_THT:D_DO-41_SOD81_P10.16mm_Horizontal, symbol Diode:1N5819
- added D7: PT1301, Package_TO_SOT_SMD:SOT-23-6_Handsoldering, symbol dcdc:PT1301
- added L1: 4.7µH, inductor:CD43, symbol pspice:INDUCTOR
- added Q3: BC817, Package_TO_SOT_SMD:SOT-23, symbol Transistor_BJT:BC817
- added Q4: IRLML6402, Package_TO_SOT_SMD:SOT-23, symbol Transistor_FET:IRLML6402
- added R18: 1K, Resistor_SMD:R_0603_1608Metric_Pad1.05x0.95mm_HandSolder, symbol Device:R
- added R19: 10K, Resistor_SMD:R_0603_1608Metric_Pad1.05x0.95mm_HandSolder, symbol Device:R
- added R20: 4K7, Resistor_SMD:R_0603_1608Metric_Pad1.05x0.95mm_HandSolder, symbol Device:R
- added R21: 27, Resistor_SMD:R_0603_1608Metric_Pad1.05x0.95mm_HandSolder, symbol Device:R
- added R22: 3M, Resistor_SMD:R_0603_1608Metric_Pad1.05x0.95mm_HandSolder, symbol Device:R
- added R23: 1M, Resistor_SMD:R_0603_1608Metric_Pad1.05x0.95mm_HandSolder, symbol Device:R
Connections:
- new net: D6.2 (A), D7.4 (LX), L1.2
- new net: D7.6 (FB), R22.2, R23.1
- new net: Q4.1 (G), R20.2, R21.1
- new net: C31.1, L1.1, Q4.3 (D)
- new net: Q3.3 (C), R21.2
- new net: Q3.1 (B), R18.2, R19.1
- new net +5V: C32.1, C33.1, D6.1 (K), D7.1 (CE), D7.5 (VDD), R22.1
- new net BAT_VDD: Q4.2 (S), R20.1
- new net GND: C31.2, C32.2, C33.2, D7.3 (GND), Q3.2 (E), R19.2, R23.2
- new net PWR_5V_ON: R18.1
