File: dcdc.sch (KiCad schematic (older format))
At the start: 14 parts, among them Q3 BC817, Q4 IRLML6402

Commit message: Сделал плату компактнее.
Parts:
- removed D6: 1N5819, Diode_THT:D_DO-41_SOD81_P10.16mm_Horizontal, symbol Diode:1N5819
- added D6: 1N4001, Diode_SMD:D_SMA_Handsoldering, symbol Diode:1N4001
Connections:
- net +5V: now also D6.1 (K)
- net at D7.4 (LX), L1.2: now also D6.2 (A)
Changed lines of the file:
@@
 $Descr A4 11693 8268
 encoding utf-8
-Sheet 5 11
+Sheet 5 12
 Title ""
 Date ""
@@
 	5300 3200 5250 3200
 Connection ~ 5250 3200
-$Comp
-L Diode:1N5819 D6
-U 1 1 5EAB9973
-P 6300 3200
-F 0 "D6" H 6300 2983 50  0000 C CNN
-F 1 "1N5819" H 6300 3074 50  0000 C CNN
-F 2 "Diode_THT:D_DO-41_SOD81_P10.16mm_Horizontal" H 6300 3025 50  0001 C CNN
-F 3 "http://www.vishay.com/docs/88525/1n5817.pdf" H 6300 3200 50  0001 C CNN
-	1    6300 3200
-	-1   0    0    1
-$EndComp
 Wire Wire Line
 	6450 3200 6500 3200
@@
 Wire Wire Line
 	6500 3200 6500 3750
+$Comp
+L Diode:1N4001 D6
+U 1 1 5EA703D8
+P 6300 3200
+F 0 "D6" H 6300 2983 50  0000 C CNN
+F 1 "1N4001" H 6300 3074 50  0000 C CNN
+F 2 "Diode_SMD:D_SMA_Handsoldering" H 6300 3025 50  0001 C CNN
+F 3 "http://www.vishay.com/docs/88503/1n4001.pdf" H 6300 3200 50  0001 C CNN
+	1    6300 3200
+	-1   0    0    1
+$EndComp
 $EndSCHEMATC

Commit message: Расставил проверенные блоки в столбец.
Connections:
- net BAT_VDD renamed VDD_BAT
Changed lines of the file:
@@
 $EndDescr
-$Comp
-L Device:R R21
-U 1 1 5EAAC84D
-P 5000 3800
-F 0 "R21" H 4800 3850 50  0000 L CNN
-F 1 "27" H 4850 3750 50  0000 L CNN
-F 2 "Resistor_SMD:R_0603_1608Metric_Pad1.05x0.95mm_HandSolder" V 4930 3800 50  0001 C CNN
-F 3 "~" H 5000 3800 50  0001 C CNN
-	1    5000 3800
-	1    0    0    -1
-$EndComp
 $Comp
 L Device:R R18
@@
 $EndComp
 Text HLabel 4700 3200 0    50   Input ~ 0
-BAT_VDD
+VDD_BAT
 $Comp
 L Transistor_FET:IRLML6402 Q4
@@
 	1    5000 3300
 	0    1    -1   0
-$EndComp
-$Comp
-L Device:R R20
-U 1 1 5EAAC4DB
-P 4750 3400
-F 0 "R20" H 4550 3450 50  0000 L CNN
-F 1 "4K7" H 4550 3350 50  0000 L CNN
-F 2 "Resistor_SMD:R_0603_1608Metric_Pad1.05x0.95mm_HandSolder" V 4680 3400 50  0001 C CNN
-F 3 "~" H 4750 3400 50  0001 C CNN
-	1    4750 3400
-	1    0    0    -1
 $EndComp
 Wire Wire Line
@@
 	-1   0    0    1
 $EndComp
+$Comp
+L Device:R R21
+U 1 1 5EAAC84D
+P 5000 3800
+F 0 "R21" H 4800 3850 50  0000 L CNN
+F 1 "27" H 4850 3750 50  0000 L CNN
+F 2 "Resistor_SMD:R_0603_1608Metric_Pad1.05x0.95mm_HandSolder" V 4930 3800 50  0001 C CNN
+F 3 "~" H 5000 3800 50  0001 C CNN
+	1    5000 3800
+	1    0    0    -1
+$EndComp
+$Comp
+L Device:R R20
+U 1 1 5EAAC4DB
+P 4750 3400
+F 0 "R20" H 4550 3450 50  0000 L CNN
+F 1 "4K7" H 4550 3350 50  0000 L CNN
+F 2 "Resistor_SMD:R_0603_1608Metric_Pad1.05x0.95mm_HandSolder" V 4680 3400 50  0001 C CNN
+F 3 "~" H 4750 3400 50  0001 C CNN
+	1    4750 3400
+	1    0    0    -1
+$EndComp
 $EndSCHEMATC
