File: mc.sch (KiCad schematic (older format))
At the start: 26 parts, among them J1 Conn_01x10_Male, U3 STM32F722ZETx, U4 W9812G6KH-6, Y1 NX3225SA-16.000M-STD-CRS-2, Y2 MC-306

Commit message: Сделал плату компактнее.
Parts:
- J1: footprint Connector_PinHeader_2.54mm:PinHeader_1x10_P2.54mm_Horizontal -> Connector_PinHeader_1.27mm:PinHeader_1x10_P1.27mm_Vertical
Changed lines of the file:
@@
 $Descr A3 16535 11693
 encoding utf-8
-Sheet 6 11
+Sheet 6 12
 Title ""
 Date ""
@@
 F 0 "J1" H 650 5050 50  0000 R CNN
 F 1 "Conn_01x10_Male" H 1200 6200 50  0000 R CNN
-F 2 "Connector_PinHeader_2.54mm:PinHeader_1x10_P2.54mm_Horizontal" H 550 5700 50  0001 C CNN
+F 2 "Connector_PinHeader_1.27mm:PinHeader_1x10_P1.27mm_Vertical" H 550 5700 50  0001 C CNN
 F 3 "~" H 550 5700 50  0001 C CNN
 	1    550  5700
